File: board-develop-raspberry-pi-kicad/board-develop-raspberry-pi-kicad.sch (KiCad schematic (older format))
At the start: 32 parts

Commit message: backup sch 1st
Parts:
- C1, C2, C3, C5, C7: renamed from C?; footprint (none) -> Capacitors_SMD:C_0805_HandSoldering
- C4: renamed from C?; footprint (none) -> Capacitors_SMD:c_elec_10x10
- C6: renamed from C?; footprint (none) -> Capacitors_SMD:c_elec_8x10
- D1, D3, D5: renamed from D?; footprint (none) -> Diodes_SMD:SOD-123
- D2, D4: renamed from D?; footprint (none) -> Diodes_SMD:SMA_Standard
- F1: renamed from F?; footprint (none) -> Fuse_Holders_and_Fuses:Fuse_SMD2920
- L1: renamed from L?; footprint (none) -> Inductors:SELF-WE-PD-XXL
- P1: renamed from P?; footprint (none) -> Connect:AK300-2
- P2: renamed from P?; footprint (none) -> Connectors_Molex:Molex_KK_6410-04
- P3: renamed from P?; value XN1 -> XN2; footprint (none) -> Connect:AK300-2
- P4: renamed from P?; footprint (none) -> Pin_Headers:Pin_Header_Straight_2x20
- Q1: renamed from Q?; footprint ~ -> TO_SOT_Packages_SMD:SOT-23
- R1, R2, R3, R4, R5, R6, R7, R8: renamed from R?; footprint (none) -> Resistors_SMD:R_0805_HandSoldering
- SP1: renamed from SP?; footprint (none) -> Buzzers_Beepers:BUZZER
- U1: renamed from U?; footprint (none) -> Housings_SOIC:SOIC-8_3.9x4.9mm_Pitch1.27mm
- U2: renamed from U?; footprint DIP-4 -> Opto-Devices:Optocoupler_SMD_HandSoldering_KPC357_LTV35x_PC357_SingleChannel
- U3: renamed from U?; footprint ~ -> TO_SOT_Packages_SMD:TO-263-5Lead
- U4: renamed from U?; footprint DIP-4 -> Devices:Optocoupler_SMD_HandSoldering_KPC357_LTV35x_PC357_SingleChannel
Connections:
- no-connect marks 0 -> 22
Other:
- moved on the sheet: C4, C5, C6, D2, D4, F1, L1, U3

Commit message: backup PCB 1st
Parts:
- removed L1: 470, Inductors:SELF-WE-PD-XXL, symbol INDUCTOR_SMALL
- added L1: INDUCTOR, Inductors:SELF-WE-PD-XXL, symbol INDUCTOR
- P1, P3: footprint Connect:AK300-2 -> conn:domino-2
- U4: footprint Devices:Optocoupler_SMD_HandSoldering_KPC357_LTV35x_PC357_SingleChannel -> Opto-Devices:Optocoupler_SMD_HandSoldering_KPC357_LTV35x_PC357_SingleChannel
Connections:
- net +5V: now also L1.2
- net at D4.1 (K), U3.2 (OUT): now also L1.1
Other:
- moved on the sheet: C1, C2, C4, C5, C6, D2, D4, D5, P2, Q1, R3, R6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
