File: board-develop-raspberry-pi-kicad/board-develop-raspberry-pi-kicad.kicad_pcb (KiCad board)
At the start: 2 copper layers, 43.9 x 65.4 mm, 36 parts, among them P1 XN1, P2 DOMINO, P3 XN2, P4 CONN_02X20, Q1 2SC1815, U1 MAX485, U2 LTV-817, U3 LM2596, U4 LTV-817

Commit message: merge develop
Routing:
- net +5V: vias 3 -> 2
- net (no net): vias 0 -> 1
Changed lines of the file:
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@@
     (links 74)
     (no_connects 0)
-    (area 50.415519 36.901 251.882049 116.198321)
+    (area 101.98456 37.406343 159.21128 107.56768)
     (thickness 1.6)
     (drawings 6)
@@
     (visible_elements 7FFCFFFF)
     (pcbplotparams
-      (layerselection 0x00030_80000001)
+      (layerselection 0x010f0_80000001)
       (usegerberextensions false)
       (excludeedgelayer true)
@@
       (outputformat 1)
       (mirror false)
-      (drillshape 1)
+      (drillshape 0)
       (scaleselection 1)
-      (outputdirectory ""))
+      (outputdirectory ../gerber/))
   )
   (net 0 "")
@@
   (gr_line (start 149.5044 41.1734) (end 105.653833 41.1734) (layer Edge.Cuts) (width 0.15))
   (gr_line (start 149.5044 41.1734) (end 149.5044 106.5784) (layer Edge.Cuts) (width 0.15))
+  (via (at 140.56868 73.77176) (size 1.1) (drill 0.7) (layers F.Cu B.Cu) (net 0))
   (segment (start 143.7894 59.5884) (end 132.04444 59.5884) (width 0.7) (layer B.Cu) (net 1))
   (segment (start 132.04444 59.5884) (end 132.00888 59.62396) (width 0.7) (layer B.Cu) (net 1))
@@
   (segment (start 140.56868 74.96556) (end 140.54328 74.99096) (width 0.6) (layer F.Cu) (net 6))
   (via (at 140.56868 72.55256) (size 1.1) (drill 0.7) (layers F.Cu B.Cu) (net 6))
-  (via (at 140.56868 73.77176) (size 1.1) (drill 0.7) (layers F.Cu B.Cu) (net 6))
   (segment (start 140.54328 74.99096) (end 140.54328 79.24292) (width 1.1) (layer F.Cu) (net 6))
   (segment (start 140.54328 79.24292) (end 140.08608 79.70012) (width 1.1) (layer F.Cu) (net 6))

Commit message: finish project version 1
Routing:
- net +5V: track 149.3 -> 117.6 mm, vias 2 -> 5
Other:
- board size 43.9 x 65.4 mm -> 43.5 x 65.4 mm
- net class Default: trace_width 1.7 -> 1.1
Changed lines of the file:
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@@
     (links 74)
     (no_connects 0)
-    (area 101.98456 37.406343 159.21128 107.56768)
+    (area 105.578832 41.098399 149.579401 106.653401)
     (thickness 1.6)
     (drawings 6)
-    (tracks 380)
+    (tracks 391)
     (zones 0)
     (modules 36)
@@
   )
   (setup
-    (last_trace_width 1.7)
+    (last_trace_width 1.1)
     (trace_clearance 0.25)
     (zone_clearance 0.508)
@@
   (net_class Default "This is the default net class."
     (clearance 0.25)
-    (trace_width 1.7)
+    (trace_width 1.1)
     (via_dia 1.1)
     (via_drill 0.7)
@@
   )
   (gr_line (start 105.65384 106.56824) (end 105.65384 41.1734) (layer Edge.Cuts) (width 0.15))
-  (gr_line (start 149.5044 106.5784) (end 105.65384 106.5784) (layer Edge.Cuts) (width 0.15))
-  (gr_line (start 149.5044 41.1734) (end 105.653833 41.1734) (layer Edge.Cuts) (width 0.15))
-  (gr_line (start 149.5044 41.1734) (end 149.5044 106.5784) (layer Edge.Cuts) (width 0.15))
+  (gr_line (start 149.17928 106.53776) (end 105.65384 106.5784) (layer Edge.Cuts) (width 0.15))
+  (gr_line (start 149.179294 41.1734) (end 105.653833 41.1734) (layer Edge.Cuts) (width 0.15))
+  (gr_line (start 149.179294 41.1734) (end 149.179294 106.553) (layer Edge.Cuts) (width 0.15))
   (via (at 140.56868 73.77176) (size 1.1) (drill 0.7) (layers F.Cu B.Cu) (net 0))
   (segment (start 143.7894 59.5884) (end 132.04444 59.5884) (width 0.7) (layer B.Cu) (net 1))
@@
   (segment (start 115.06708 98.10242) (end 121.07672 98.10242) (width 0.7) (layer F.Cu) (net 5))
   (segment (start 121.07672 98.10242) (end 123.26112 95.91802) (width 0.7) (layer F.Cu) (net 5))
-  (segment (start 146.3294 51.9684) (end 148.86329 54.50229) (width 0.45) (layer B.Cu) (net 6))
-  (segment (start 141.45768 75.90536) (end 140.54328 74.99096) (width 0.45) (layer B.Cu) (net 6))
-  (segment (start 148.86329 54.50229) (end 148.86329 98.54795) (width 0.45) (layer B.Cu) (net 6))
-  (segment (start 147.02028 100.39096) (end 142.54988 100.39096) (width 0.45) (layer B.Cu) (net 6))
-  (segment (start 142.54988 100.39096) (end 141.45768 99.29876) (width 0.45) (layer B.Cu) (net 6))
-  (segment (start 148.86329 98.54795) (end 147.02028 100.39096) (width 0.45) (layer B.Cu) (net 6))
-  (segment (start 141.45768 99.29876) (end 141.45768 75.90536) (width 0.45) (layer B.Cu) (net 6))
+  (segment (start 119.71528 73.72096) (end 119.71528 72.5772) (width 1.1) (layer B.Cu) (net 6))
+  (segment (start 119.71528 72.5772) (end 119.73992 72.55256) (width 1.1) (layer B.Cu) (net 6))
+  (segment (start 119.76608 71.38416) (end 119.76608 72.5264) (width 1.1) (layer F.Cu) (net 6))
+  (segment (start 119.76608 72.5264) (end 119.73992 72.55256) (width 1.1) (layer F.Cu) (net 6))
+  (segment (start 119.76608 71.38416) (end 119.76608 72.5264) (width 1.1) (layer B.Cu) (net 6))
+  (segment (start 119.76608 72.5264) (end 119.73992 72.55256) (width 1.1) (layer B.Cu) (net 6))
+  (via (at 119.71528 73.72096) (size 1.1) (drill 0.7) (layers F.Cu B.Cu) (net 6))
+  (via (at 119.76608 71.38416) (size 1.1) (drill 0.7) (layers F.Cu B.Cu) (net 6))
+  (segment (start 146.3294 49.4284) (end 146.3294 48.51908) (width 1.1) (layer B.Cu) (net 6))
+  (segment (start 146.3294 48.51908) (end 145.06448 47.25416) (width 1.1) (layer B.Cu) (net 6))
+  (segment (start 140.64488 44.61256) (end 139.07008 44.61256) (width 1.1) (layer B.Cu) (net 6))
+  (segment (start 145.06448 47.25416) (end 143.28648 47.25416) (width 1.1) (layer B.Cu) (net 6))
+  (segment (start 143.28648 47.25416) (end 140.64488 44.61256) (width 1.1) (layer B.Cu) (net 6))
+  (segment (start 139.07008 44.61256) (end 119.76608 63.91656) (width 1.1) (layer B.Cu) (net 6))
+  (segment (start 119.76608 63.91656) (end 119.76608 72.5264) (width 1.1) (layer B.Cu) (net 6))
+  (segment (start 119.73992 70.01256) (end 119.73992 72.55256) (width 1.3) (layer F.Cu) (net 6))
+  (segment (start 119.73992 72.55256) (end 119.73992 75.52944) (width 1.3) (layer F.Cu) (net 6))
+  (via (at 119.73992 72.55256) (size 1.1) (drill 0.7) (layers F.Cu B.Cu) (net 6))
   (segment (start 140.56868 72.55256) (end 140.56868 74.96556) (width 0.45) (layer B.Cu) (net 6))
   (segment (start 140.56868 74.96556) (end 140.54328 74.99096) (width 0.7) (layer B.Cu) (net 6))
@@
   (segment (start 137.16508 75.52944) (end 140.08608 78.45044) (width 1.1) (layer F.Cu) (net 6))
   (segment (start 140.08608 78.45044) (end 140.08608 79.70012) (width 1.1) (layer F.Cu) (net 6))
-  (segment (start 119.73992 70.01256) (end 119.73992 75.52944) (width 1.3) (layer F.Cu) (net 6))
   (segment (start 119.96928 74.99096) (end 119.96928 75.52944) (width 1.3) (layer F.Cu) (net 6))
   (segment (start 119.96928 75.30008) (end 119.96928 74.99096) (width 1.3) (layer F.Cu) (net 6))
@@
   (segment (start 109.0522 93.99028) (end 109.0522 88.7492) (width 1.7) (layer F.Cu) (net 15))
   (segment (start 109.0522 88.7492) (end 108.2886 87.9856) (width 1.7) (layer F.Cu) (net 15))
-  (segment (start 137.36828 49.56556) (end 136.63168 49.56556) (width 0.7) (layer B.Cu) (net 16))
-  (segment (start 136.63168 49.56556) (end 136.17448 49.10836) (width 0.7) (layer B.Cu) (net 16))
+  (segment (start 136.328988 49.304085) (end 136.328988 49.262868) (width 0.7) (layer B.Cu) (net 16))
+  (segment (start 136.590463 49.56556) (end 136.328988 49.304085) (width 0.7) (layer B.Cu) (net 16))
+  (via (at 136.328988 49.262868) (size 1.1) (drill 0.7) (layers F.Cu B.Cu) (net 16))
+  (segment (start 137.36828 49.56556) (end 136.590463 49.56556) (width 0.7) (layer B.Cu) (net 16))
   (segment (start 138.51128 49.590956) (end 137.393676 49.590956) (width 0.7) (layer B.Cu) (net 16))
   (segment (start 137.393676 49.590956) (end 137.36828 49.56556) (width 0.7) (layer B.Cu) (net 16))
-  (via (at 136.17448 49.10836) (size 1.1) (drill 0.7) (layers F.Cu B.Cu) (net 16))
   (via (at 137.36828 49.56556) (size 1.1) (drill 0.7) (layers F.Cu B.Cu) (net 16))
   (segment (start 135.38708 73.49236) (end 136.58088 73.49236) (width 1.1) (layer F.Cu) (net 16))
@@
   (segment (start 128.85928 66.86296) (end 130.30928 66.86296) (width 0.6) (layer F.Cu) (net 45))
   (segment (start 130.30928 66.86296) (end 131.77012 68.3238) (width 0.6) (layer F.Cu) (net 45))
+  (zone (net 1) (net_name GND) (layer B.Cu) (hatch edge 0.508)
+    (connect_pads (clearance 0.508))
+    (min_thickness 0.3)
+    (fill yes (arc_segments 16) (thermal_gap 0.508) (thermal_bridge_width 0.508))
+    (polygon
+      (pts
+        (xy 105.64368 41.18356) (xy 149.17928 41.18356) (xy 149.17928 106.53776) (xy 105.66908 106.53776) (xy 105.64368 106.53776)
+      )
+    )
+  )
   (zone (net 1) (net_name GND) (layer F.Cu) (hatch edge 0.508)
     (connect_pads (clearance 0.508))
@@
     (polygon
       (pts
-        (xy 105.66908 41.18356) (xy 149.50948 41.18356) (xy 149.50948 106.56316) (xy 105.64368 106.56316) (xy 105.64368 41.18356)
+        (xy 105.64368 41.18356) (xy 149.17928 41.18356) (xy 149.17928 106.53776) (xy 105.64368 106.53776)
       )
     )
-  )
-  (zone (net 1) (net_name GND) (layer B.Cu) (hatch edge 0.508)
-    (connect_pads (clearance 0.508))
-    (min_thickness 0.3)
-    (fill yes (arc_segments 16) (thermal_gap 0.508) (thermal_bridge_width 0.508))
-    (polygon
-      (pts
-        (xy 105.64368 41.18356) (xy 149.50948 41.18356) (xy 149.50948 106.56316) (xy 105.64368 106.56316)
-      )
-    )
